File: _saved_kicad.sch (KiCad schematic (older format))
At the start: 10 parts, among them J1 KF350, J2 ESP8266, K1 JRC-21F(4100)

Commit message: v1.1
Parts:
- C1: footprint footprints:C10uF -> footprints:C_1206_3216Metric
- D1: renamed from D?; footprint (none) -> footprints:D_SMA
- PS1: renamed from PS?; footprint (none) -> footprints:0103YN
- Q1: renamed from Q?; footprint (none) -> footprints:SOT-23
- R1: renamed from R?; footprint (none) -> footprints:R_0805_2012Metric
- U1: renamed from U?; footprint (none) -> footprints:SOT-223
Changed lines of the file:
@@
 F 0 "C1" H 5450 3050 50  0000 C CNN
 F 1 "10uF" H 5375 2876 50  0000 C CNN
-F 2 "footprints:C10uF" H 5350 3000 50  0001 C CNN
+F 2 "footprints:C_1206_3216Metric" H 5350 3000 50  0001 C CNN
 F 3 "" H 5350 3000 50  0001 C CNN
 	1    5400 3000
@@
 	6550 3350 6550 3600
 $Comp
-L local:LD1117V33C U?
+L local:LD1117V33C U1
 U 1 1 62C9D78F
 P 4850 3650
-F 0 "U?" H 4850 3851 39  0000 C CNN
+F 0 "U1" H 4850 3851 39  0000 C CNN
 F 1 "LD1117V33C" H 4850 3776 39  0000 C CNN
-F 2 "" H 5000 3750 50  0001 C CNN
+F 2 "footprints:SOT-223" H 5000 3750 50  0001 C CNN
 F 3 "" H 5000 3750 50  0001 C CNN
 	1    4850 3650
@@
 $EndComp
 $Comp
-L power:GND #PWR?
+L power:GND #PWR03
 U 1 1 62C9DB5E
 P 4850 4000
-F 0 "#PWR?" H 4850 3750 50  0001 C CNN
+F 0 "#PWR03" H 4850 3750 50  0001 C CNN
 F 1 "GND" H 4855 3835 39  0000 C CNN
 F 2 "" H 4850 4000 50  0001 C CNN
@@
 	5250 3000 5250 3650
 $Comp
-L local:MMBT4403 Q?
+L local:MMBT4403 Q1
 U 1 1 62C9EFB8
 P 6950 2650
-F 0 "Q?" H 7050 2800 50  0000 C CNN
+F 0 "Q1" H 7050 2800 50  0000 C CNN
 F 1 "MMBT4403" H 6950 2450 50  0000 C CNN
-F 2 "" V 6950 2650 50  0001 C CNN
+F 2 "footprints:SOT-23" V 6950 2650 50  0001 C CNN
 F 3 "" V 6950 2650 50  0001 C CNN
 	1    6950 2650
@@
 $EndComp
 $Comp
-L power:+3V3 #PWR?
+L power:+3V3 #PWR09
 U 1 1 62C9F699
 P 6450 4200
-F 0 "#PWR?" H 6450 4050 50  0001 C CNN
+F 0 "#PWR09" H 6450 4050 50  0001 C CNN
 F 1 "+3V3" H 6465 4373 50  0000 C CNN
 F 2 "" H 6450 4200 50  0001 C CNN
@@
 Connection ~ 5250 3650
 $Comp
-L power:+3V3 #PWR?
+L power:+3V3 #PWR06
 U 1 1 62C9FF50
 P 5250 3850
-F 0 "#PWR?" H 5250 3700 50  0001 C CNN
+F 0 "#PWR06" H 5250 3700 50  0001 C CNN
 F 1 "+3V3" H 5265 4023 50  0000 C CNN
 F 2 "" H 5250 3850 50  0001 C CNN
@@
 	6450 2700 6750 2700
 $Comp
-L power:GND #PWR?
+L power:GND #PWR010
 U 1 1 62CA220E
 P 7350 2750
-F 0 "#PWR?" H 7350 2500 50  0001 C CNN
+F 0 "#PWR010" H 7350 2500 50  0001 C CNN
 F 1 "GND" H 7355 2585 39  0000 C CNN
 F 2 "" H 7350 2750 50  0001 C CNN
@@
 	7350 2700 7350 2750
 $Comp
-L local:0102YN PS?
+L local:0102YN PS1
 U 1 1 62CA3141
 P 3900 3750
-F 0 "PS?" H 3716 3996 50  0000 C CNN
+F 0 "PS1" H 3716 3996 50  0000 C CNN
 F 1 "0102YN" H 4000 3500 50  0000 C CNN
-F 2 "" H 3900 3600 50  0001 C CNN
+F 2 "footprints:0103YN" H 3900 3600 50  0001 C CNN
 F 3 "" H 3900 3600 50  0001 C CNN
 	1    3900 3750
@@
 	2800 3800 3550 3800
 $Comp
-L local:R_1k R?
+L local:R_1k R1
 U 1 1 62CA9825
 P 6600 2350
-F 0 "R?" V 6514 2298 50  0000 C CNN
+F 0 "R1" V 6514 2298 50  0000 C CNN
 F 1 "1K" V 6698 2366 50  0000 C CNN
-F 2 "" H 6600 2350 50  0001 C CNN
+F 2 "footprints:R_0805_2012Metric" H 6600 2350 50  0001 C CNN
 F 3 "" H 6600 2350 50  0001 C CNN
 	1    6600 2350
@@
 	6350 2350 6450 2350
 $Comp
-L local:Diode D?
+L local:Diode D1
 U 1 1 62CABD93
 P 6050 3300
-F 0 "D?" H 6050 3200 50  0000 C CNN
+F 0 "D1" H 6050 3200 50  0000 C CNN
 F 1 "Diode" H 6032 3412 50  0000 C CNN
-F 2 "" H 6050 3300 50  0001 C CNN
+F 2 "footprints:D_SMA" H 6050 3300 50  0001 C CNN
 F 3 "" H 6050 3300 50  0001 C CNN
 	1    6050 3300
@@
 	6450 3300 6450 2700
 $Comp
-L power:+3V3 #PWR?
+L power:+3V3 #PWR08
 U 1 1 62CAD1B4
 P 5800 3400
-F 0 "#PWR?" H 5800 3250 50  0001 C CNN
+F 0 "#PWR08" H 5800 3250 50  0001 C CNN
 F 1 "+3V3" H 5815 3573 50  0000 C CNN
 F 2 "" H 5800 3400 50  0001 C CNN
