File: smart-movement-sensor/smart-movement-sensor.sch (KiCad schematic (older format))
At the start: 17 parts

Commit message: New features
Parts:
- added D1: led, fooprint:LED_0805, symbol local:led
- added Q2: 2n2222, fooprint:SOT-23, symbol local:2n2222
- added R2: 200R, fooprint:R_0805_2012Metric, symbol local:R_1k
- added R4: 1R, fooprint:R_0805_2012Metric, symbol local:R_1k
- added R6: 7.5R, fooprint:R_0805_2012Metric, symbol local:R_1k
- C1: renamed from C?; value 10uF -> 1uF; footprint (none) -> fooprint:C_1206_3216Metric
- D2: renamed from D?; footprint (none) -> fooprint:D_SMA
- J1: renamed from J?; footprint (none) -> fooprint:ESP8266
- Q1, Q3, Q4: renamed from U?; footprint (none) -> fooprint:SOT-23
- R1, R3, R5, R7, R8: renamed from R?; value R_1k -> 1k; footprint (none) -> fooprint:R_0805_2012Metric
- S1: renamed from S?; footprint (none) -> fooprint:SW_Tactile
- U1: renamed from U?; value usb-micro-B -> USB micro B; footprint (none) -> Connector_USB:USB_Micro-B_Wuerth_614105150721_Vertical
- U2: renamed from U?; value movement-sensor -> movement sensor; footprint (none) -> fooprint:MS_3pins
- U3: renamed from U?; footprint (none) -> fooprint:SOP14
- U4: renamed from U?; footprint (none) -> fooprint:SOT-223
- U5: renamed from U?; footprint (none) -> fooprint:battery_603040
Connections:
- net GND: now also R4.2, R6.2; no longer Q1.2 (E), U1.5 (GND)
- net at D2.2 (A), R1.1, U1.1 (VBUS): now also D1.2 (A)
- new net: D1.1 (K), R2.2
- new net: Q2.3 (C), R2.1
- new net: Q2.1 (B), R4.1
- new net Earth: Q1.2 (E), Q2.2 (E), R6.1, U1.5 (GND)
Other:
- moved on the sheet: C1, D2, J1, Q1, Q3, Q4, R1, R3, R5, R7, R8, S1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
