File: smart-movement-sensor/smart-movement-sensor.kicad_sch (KiCad schematic)
At the start: 22 parts, among them J1 ESP8266, Q1 2n2222, Q2 2n2222, Q3 Q_PNP_CBE, Q4 2n2222, U1 USB micro B, U2 battery, U3 sensor, U4 SN74AHC1G86DBVR

Commit message: Update projects designs
Parts:
- removed Q1: 2n2222, symbol Device:Q_NPN_CBE
- removed R2: 5R, symbol Device:R_Small_US
- removed U4: SN74AHC1G86DBVR, footprints:SOP14, symbol local:SN74AHC1G86DBVR
- added U2: 74HC86, symbol 74xx:74HC86
- R1: value 1K -> 100K
- renumbered Q2 to Q1, Q3 to Q2, Q4 to Q3, R3 to R2, R4 to R3, R5 to R4, R6 to R5, R7 to R6, U2 to U3, U3 to U4
Connections:
- net GND: now also R1.1, U2.7 (GND)
- net reset signal: no longer Q3.2 (B)
- net sensor signal: now also U2.4
- net sensor signal delayed: now also U2.5
- net XVCC: now reaches D1.1 (K), D2.2 (A), Q1.1 (C), R3.1, U3.1 (+)
- net XVCC: now also U2.1, U2.14 (VCC)
- net Charge bat: now reaches D1.2 (A), U1.1 (VBUS)
- net Charge bat: now also R1.2, U2.2; no longer R1.1
- net at Q1.2 (B): now also U2.3
- new net: Q3.2 (B), U2.6
Other:
- note added: "XOR power supply"
- moved on the sheet: D1, R5
